File: hw/Schematics/Schematic_1/Schematic_1.kicad_sch (KiCad schematic)
At the start: 1 part

Commit message: XL6009
Parts:
- added U?: ABX00027, MODULE_ABX00027, symbol library_1:ABX00027
- added U?: VL53L1CXV0FY1, Sensor_Distance:ST_VL53L1x, symbol Sensor_Distance:VL53L1CXV0FY1
Connections:
- new net: U?.13 (~{RESET}), U?.18 (~{RESET})
- new net: U?.14 (GND), U?.19 (GND)
- new net: U?.12 (GND), U?.3 (GND), U?.4 (GND), U?.6 (GND)
Changed lines of the file:
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@@
 (kicad_sch (version 20211123) (generator eeschema)
   (paper "A4")
+  (symbol (lib_id "library_1:ABX00027") (at 175.26 100.33 0) (unit 1)
+    (in_bom yes) (on_board yes) (fields_autoplaced)
+    (property "Reference" "U?" (id 0) (at 175.26 69.85 0))
+    (property "Value" "ABX00027" (id 1) (at 175.26 72.39 0))
+    (property "Footprint" "MODULE_ABX00027" (id 2) (at 175.26 100.33 0)
+      (effects (font (size 1.27 1.27)) (justify left bottom) hide)
+    )
+    (property "Datasheet" "" (id 3) (at 175.26 100.33 0)
+      (effects (font (size 1.27 1.27)) (justify left bottom) hide)
+    )
+    (property "AVAILABILITY" "Unavailable" (id 4) (at 175.26 100.33 0)
+      (effects (font (size 1.27 1.27)) (justify left bottom) hide)
+    )
+    (property "MP" "ABX00027" (id 5) (at 175.26 100.33 0)
+      (effects (font (size 1.27 1.27)) (justify left bottom) hide)
+    )
+    (property "DIGIKEY-PURCHASE-URL" "https://snapeda.com/shop?store=DigiKey&id=3949339" (id 6) (at 149.86 133.35 0)
+      (effects (font (size 1.27 1.27)) (justify left bottom) hide)
+    )
+    (property "PACKAGE" "None" (id 7) (at 175.26 100.33 0)
+      (effects (font (size 1.27 1.27)) (justify left bottom) hide)
+    )
+    (property "PRICE" "None" (id 8) (at 175.26 100.33 0)
+      (effects (font (size 1.27 1.27)) (justify left bottom) hide)
+    )
+    (property "MF" "Arduino" (id 9) (at 175.26 100.33 0)
+      (effects (font (size 1.27 1.27)) (justify left bottom) hide)
+    )
+    (property "DESCRIPTION" "ATSAMD21G18A Arduino Nano 33 IoT SAM D ARM® Cortex®-M0+ MCU 32-Bit Embedded Evaluation Board" (id 10) (at 148.59 130.81 0)
+      (effects (font (size 1.27 1.27)) (justify left bottom) hide)
+    )
+    (pin "1")
+    (pin "10")
+    (pin "11")
+    (pin "12")
+    (pin "13")
+    (pin "14")
+    (pin "15")
+    (pin "16")
+    (pin "17")
+    (pin "18")
+    (pin "19")
+    (pin "2")
+    (pin "20")
+    (pin "21")
+    (pin "22")
+    (pin "23")
+    (pin "24")
+    (pin "25")
+    (pin "26")
+    (pin "27")
+    (pin "28")
+    (pin "29")
+    (pin "3")
+    (pin "30")
+    (pin "4")
+    (pin "5")
+    (pin "6")
+    (pin "7")
+    (pin "8")
+    (pin "9")
+  )
   (symbol (lib_id "Driver_Motor:DRV8871DDA") (at 115.57 104.14 0) (unit 1)
     (in_bom yes) (on_board yes) (fields_autoplaced)
@@
     (pin "9")
   )
+  (symbol (lib_id "Sensor_Distance:VL53L1CXV0FY1") (at 233.68 90.17 0) (unit 1)
+    (in_bom yes) (on_board yes) (fields_autoplaced)
+    (property "Reference" "U?" (id 0) (at 242.57 88.8999 0)
+      (effects (font (size 1.27 1.27)) (justify left))
+    )
+    (property "Value" "VL53L1CXV0FY1" (id 1) (at 242.57 91.4399 0)
+      (effects (font (size 1.27 1.27)) (justify left))
+    )
+    (property "Footprint" "Sensor_Distance:ST_VL53L1x" (id 2) (at 250.825 104.14 0)
+      (effects (font (size 1.27 1.27)) hide)
+    )
+    (property "Datasheet" "https://www.st.com/resource/en/datasheet/vl53l1x.pdf" (id 3) (at 236.22 90.17 0)
+      (effects (font (size 1.27 1.27)) hide)
+    )
+    (pin "1")
+    (pin "10")
+    (pin "11")
+    (pin "12")
+    (pin "2")
+    (pin "3")
+    (pin "4")
+    (pin "5")
+    (pin "6")
+    (pin "7")
+    (pin "8")
+    (pin "9")
+  )
   (sheet_instances
     (path "/" (page "1"))
   )
   (symbol_instances
+    (path "/22e86342-4471-4f0e-8e0a-cd51b4974fbe"
+      (reference "U?") (unit 1) (value "ABX00027") (footprint "MODULE_ABX00027")
+    )
     (path "/3633bc1f-4dc8-49cd-8d7f-d808b6df04b6"
       (reference "U?") (unit 1) (value "DRV8871DDA") (footprint "Package_SO:Texas_HTSOP-8-1EP_3.9x4.9mm_P1.27mm_EP2.95x4.9mm_Mask2.4x3.1mm_ThermalVias")
     )
+    (path "/62d56b7c-83bc-4c5e-9c1b-9248d18a2421"
+      (reference "U?") (unit 1) (value "VL53L1CXV0FY1") (footprint "Sensor_Distance:ST_VL53L1x")
+    )
   )

Commit message: sharp58
Parts:
- added U?: XL6009_BOOST, symbol library_1:XL6009_BOOST
- added U? (x4): VL53L1CXV0FY1, Sensor_Distance:ST_VL53L1x, symbol Sensor_Distance:VL53L1CXV0FY1
- added U?: Sharp58_optic_switch, symbol library_1:Sharp58_optic_switch
Connections:
- new net: U?.12 (GND), U?.3 (GND), U?.4 (GND), U?.6 (GND) (x4)
Changed lines of the file:
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@@
+    (pin "9")
+  )
+  (symbol (lib_id "library_1:XL6009_BOOST") (at 115.57 123.19 0) (unit 1)
+    (in_bom yes) (on_board yes) (fields_autoplaced)
+    (property "Reference" "U?" (id 0) (at 115.57 120.65 0))
+    (property "Value" "XL6009_BOOST" (id 1) (at 115.57 123.19 0))
+    (property "Footprint" "" (id 2) (at 115.57 123.19 0)
+      (effects (font (size 1.27 1.27)) hide)
+    )
+    (property "Datasheet" "" (id 3) (at 115.57 123.19 0)
+      (effects (font (size 1.27 1.27)) hide)
+    )
+    (pin "")
+    (pin "")
+    (pin "")
+    (pin "")
+  )
+  (symbol (lib_id "Sensor_Distance:VL53L1CXV0FY1") (at 231.14 15.24 0) (unit 1)
+    (in_bom yes) (on_board yes) (fields_autoplaced)
+    (property "Reference" "U?" (id 0) (at 240.03 13.9699 0)
+      (effects (font (size 1.27 1.27)) (justify left))
+    )
+    (property "Value" "VL53L1CXV0FY1" (id 1) (at 240.03 16.5099 0)
+      (effects (font (size 1.27 1.27)) (justify left))
+    )
+    (property "Footprint" "Sensor_Distance:ST_VL53L1x" (id 2) (at 248.285 29.21 0)
+      (effects (font (size 1.27 1.27)) hide)
+    )
+    (property "Datasheet" "https://www.st.com/resource/en/datasheet/vl53l1x.pdf" (id 3) (at 233.68 15.24 0)
+      (effects (font (size 1.27 1.27)) hide)
+    )
+    (pin "1")
+    (pin "10")
+    (pin "11")
+    (pin "12")
+    (pin "2")
+    (pin "3")
+    (pin "4")
+    (pin "5")
+    (pin "6")
+    (pin "7")
+    (pin "8")
     (pin "9")
   )
@@
     (pin "8")
     (pin "9")
+  )
+  (symbol (lib_id "Sensor_Distance:VL53L1CXV0FY1") (at 231.14 52.07 0) (unit 1)
+    (in_bom yes) (on_board yes) (fields_autoplaced)
+    (property "Reference" "U?" (id 0) (at 240.03 50.7999 0)
+      (effects (font (size 1.27 1.27)) (justify left))
+    )
+    (property "Value" "VL53L1CXV0FY1" (id 1) (at 240.03 53.3399 0)
+      (effects (font (size 1.27 1.27)) (justify left))
+    )
+    (property "Footprint" "Sensor_Distance:ST_VL53L1x" (id 2) (at 248.285 66.04 0)
+      (effects (font (size 1.27 1.27)) hide)
+    )
+    (property "Datasheet" "https://www.st.com/resource/en/datasheet/vl53l1x.pdf" (id 3) (at 233.68 52.07 0)
+      (effects (font (size 1.27 1.27)) hide)
+    )
+    (pin "1")
+    (pin "10")
+    (pin "11")
+    (pin "12")
+    (pin "2")
+    (pin "3")
+    (pin "4")
+    (pin "5")
+    (pin "6")
+    (pin "7")
+    (pin "8")
+    (pin "9")
+  )
+  (symbol (lib_id "Sensor_Distance:VL53L1CXV0FY1") (at 233.68 134.62 0) (unit 1)
+    (in_bom yes) (on_board yes) (fields_autoplaced)
+    (property "Reference" "U?" (id 0) (at 242.57 133.3499 0)
+      (effects (font (size 1.27 1.27)) (justify left))
+    )
+    (property "Value" "VL53L1CXV0FY1" (id 1) (at 242.57 135.8899 0)
+      (effects (font (size 1.27 1.27)) (justify left))
+    )
+    (property "Footprint" "Sensor_Distance:ST_VL53L1x" (id 2) (at 250.825 148.59 0)
+      (effects (font (size 1.27 1.27)) hide)
+    )
+    (property "Datasheet" "https://www.st.com/resource/en/datasheet/vl53l1x.pdf" (id 3) (at 236.22 134.62 0)
+      (effects (font (size 1.27 1.27)) hide)
+    )
+    (pin "1")
+    (pin "10")
+    (pin "11")
+    (pin "12")
+    (pin "2")
+    (pin "3")
+    (pin "4")
+    (pin "5")
+    (pin "6")
+    (pin "7")
+    (pin "8")
+    (pin "9")
+  )
+  (symbol (lib_id "Sensor_Distance:VL53L1CXV0FY1") (at 270.51 46.99 0) (unit 1)
+    (in_bom yes) (on_board yes) (fields_autoplaced)
+    (property "Reference" "U?" (id 0) (at 279.4 45.7199 0)
+      (effects (font (size 1.27 1.27)) (justify left))
+    )
+    (property "Value" "VL53L1CXV0FY1" (id 1) (at 279.4 48.2599 0)
+      (effects (font (size 1.27 1.27)) (justify left))
+    )
+    (property "Footprint" "Sensor_Distance:ST_VL53L1x" (id 2) (at 287.655 60.96 0)
+      (effects (font (size 1.27 1.27)) hide)
+    )
+    (property "Datasheet" "https://www.st.com/resource/en/datasheet/vl53l1x.pdf" (id 3) (at 273.05 46.99 0)
+      (effects (font (size 1.27 1.27)) hide)
+    )
+    (pin "1")
+    (pin "10")
+    (pin "11")
+    (pin "12")
+    (pin "2")
+    (pin "3")
+    (pin "4")
+    (pin "5")
+    (pin "6")
+    (pin "7")
+    (pin "8")
+    (pin "9")
+  )
+  (symbol (lib_id "library_1:Sharp58_optic_switch") (at 172.72 134.62 0) (unit 1)
+    (in_bom yes) (on_board yes) (fields_autoplaced)
+    (property "Reference" "U?" (id 0) (at 172.72 132.08 0))
+    (property "Value" "Sharp58_optic_switch" (id 1) (at 172.72 134.62 0))
+    (property "Footprint" "" (id 2) (at 172.72 134.62 0)
+      (effects (font (size 1.27 1.27)) hide)
+    )
+    (property "Datasheet" "" (id 3) (at 172.72 134.62 0)
+      (effects (font (size 1.27 1.27)) hide)
+    )
+    (pin "")
+    (pin "")
+    (pin "")
+    (pin "")
   )
   (sheet_instances
@@
       (reference "U?") (unit 1) (value "ABX00027") (footprint "MODULE_ABX00027")
     )
+    (path "/32e588e5-b446-4594-aa05-501c69962c80"
+      (reference "U?") (unit 1) (value "XL6009_BOOST") (footprint "")
+    )
+    (path "/35c3b0d4-2187-4274-a53d-a1d41d2197dd"
+      (reference "U?") (unit 1) (value "VL53L1CXV0FY1") (footprint "Sensor_Distance:ST_VL53L1x")
+    )
     (path "/3633bc1f-4dc8-49cd-8d7f-d808b6df04b6"
       (reference "U?") (unit 1) (value "DRV8871DDA") (footprint "Package_SO:Texas_HTSOP-8-1EP_3.9x4.9mm_P1.27mm_EP2.95x4.9mm_Mask2.4x3.1mm_ThermalVias")
@@
       (reference "U?") (unit 1) (value "VL53L1CXV0FY1") (footprint "Sensor_Distance:ST_VL53L1x")
     )
-  )
+    (path "/79f95f95-dc40-4d71-af05-5fb27436421e"
+      (reference "U?") (unit 1) (value "VL53L1CXV0FY1") (footprint "Sensor_Distance:ST_VL53L1x")
+    )
+    (path "/a357748c-aeb1-4822-afaa-263d5d7d5e7e"
+      (reference "U?") (unit 1) (value "VL53L1CXV0FY1") (footprint "Sensor_Distance:ST_VL53L1x")
+    )
+    (path "/aa1684cb-fbdc-450d-887c-6026d3066c7e"
+      (reference "U?") (unit 1) (value "VL53L1CXV0FY1") (footprint "Sensor_Distance:ST_VL53L1x")
+    )
+    (path "/b6d94b8e-1631-4ff1-a244-4f1114d1ce2d"
+      (reference "U?") (unit 1) (value "Sharp58_optic_switch") (footprint "")
+    )
+  )

Commit message: Sharp582
Parts:
- removed U?: Sharp58_optic_switch, symbol library_1:Sharp58_optic_switch
- added BT?: Battery_Cell, symbol Device:Battery_Cell
- added U?: Switchregulator_step-down_0.8V_-_17_V, symbol library_1:Switchregulator_step-down_0.8V_-_17_V
- added U?: Sharp58_optic_switch, symbol library_1:Sharp58_optic_switch
Other:
- moved on the sheet: U?

Commit message: Schema version 1
Parts:
- removed BT?: Battery_Cell, symbol Device:Battery_Cell
- removed U? (x5): VL53L1CXV0FY1, Sensor_Distance:ST_VL53L1x, symbol Sensor_Distance:VL53L1CXV0FY1
- added BT?: Battery_Cell, symbol Device:Battery_Cell
- added M?: Motor_DC, symbol Motor:Motor_DC
- added R1, R2: R, symbol Device:R
- added Styrservo: Motor_Servo, symbol Motor:Motor_Servo
- added U? (x5): VL53L1CXV0FY1, Sensor_Distance:ST_VL53L1x, symbol Sensor_Distance:VL53L1CXV0FY1
- gave numbers to parts that had none: 1
Connections:
- net RÖD: now reaches 3.3V_Buck. (VO+)
- net RÖD: now also R1.1, R2.2, Styrservo.2 (+), U?.11 (AVDD), U?.11 (AVDD), U?.11 (AVDD), U?.11 (AVDD), U?.11 (AVDD)
- net at U?.10 (A6): now also U?.5 (XSHUT)
- net at U?.11 (A7): now also U?.5 (XSHUT)
- net GND: now reaches U?.14 (GND), U?.19 (GND)
- net GND: now also 3.3V_Buck. (VO+), U?. (Kollektor), U?. (OUT-), U?.1 (GND), U?.7 (GND), U?.9 (GND), BT?.2 (-), R2.1, Styrservo.3 (-), U?.12 (GND), U?.12 (GND), U?.12 (GND), U?.12 (GND), U?.12 (GND), U?.3 (GND), U?.3 (GND), U?.3 (GND), U?.3 (GND), U?.3 (GND), U?.4 (GND), U?.4 (GND), U?.4 (GND), U?.4 (GND), U?.4 (GND), U?.6 (GND), U?.6 (GND), U?.6 (GND), U?.6 (GND), U?.6 (GND)
- net at U?.15 (VIN): now also U?. (OUT-), U?.5 (VM)
- net at U?.23 (D5/PWM): now also U?.3 (IN1)
- net at U?.24 (D6/PWM): now also U?.2 (IN2)
- net GUL: now reaches U?.27 (D9/PWM)
- net GUL: now also Styrservo.1 (PWM)
- net at U?.5 (A1): now also U?.5 (XSHUT)
- net at U?.6 (A2): now also U?.5 (XSHUT)
- net at U?.7 (A3): now also U?.5 (XSHUT)
- net at U?.8 (A4/SDA): now also U?.9 (SDA), U?.9 (SDA), U?.9 (SDA), U?.9 (SDA), U?.9 (SDA)
- net at U?.9 (A5/SCL): now also U?.10 (SCL), U?.10 (SCL), U?.10 (SCL), U?.10 (SCL)
- net at U?.6 (OUT1): now also M?.1 (+)
- net at U?.8 (OUT2): now also M?.2 (-)
- new net: 3.3V_Buck. (VO+), BT?.1 (+), U?. (OUT-)
- new net: R1.2, U?. (Kollektor)
Other:
- moved on the sheet: 3.3V_Buck, U?

Commit message: allman
Connections:
- net GND: no longer R2.1
- new net: 3.3V_Buck. (VO+), BT?.1 (+), U?. (OUT-)
- new net: R2.1, U?. (Kollektor)
Other:
- moved on the sheet: R2
Changed lines of the file:
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@@
 (kicad_sch (version 20211123) (generator eeschema)
   (paper "A4")
+  (junction (at 129.54 109.22) (diameter 0) (color 0 0 0 0)
+  )
   (junction (at 54.61 -21.59) (diameter 0) (color 0 0 0 0)
   )
@@
   (junction (at 77.47 39.37) (diameter 0) (color 0 0 0 0)
   )
-  (junction (at 121.92 85.09) (diameter 0) (color 0 0 0 0)
-  )
   (wire (pts (xy 199.39 39.37) (xy 199.39 48.26))
     (stroke (width 0) (type default) (color 0 0 0 0))
@@
     (stroke (width 0) (type default) (color 0 0 0 0))
   )
-  (wire (pts (xy 132.08 85.09) (xy 132.08 109.22))
+  (wire (pts (xy 129.54 109.22) (xy 132.08 109.22))
     (stroke (width 0) (type default) (color 0 0 0 0))
   )
@@
     (stroke (width 0) (type default) (color 0 0 0 0))
   )
+  (wire (pts (xy 129.54 87.63) (xy 129.54 109.22))
+    (stroke (width 0) (type default) (color 0 0 0 0))
+  )
   (wire (pts (xy 187.96 0) (xy 223.52 0))
     (stroke (width 0) (type default) (color 0 0 0 0))
   )
-  (wire (pts (xy 121.92 85.09) (xy 124.46 85.09))
+  (wire (pts (xy 121.92 85.09) (xy 121.92 87.63))
     (stroke (width 0) (type default) (color 0 0 0 0))
   )
@@
     (stroke (width 0) (type default) (color 0 0 0 0))
   )
-  (wire (pts (xy 121.92 85.09) (xy 121.92 93.98))
-    (stroke (width 0) (type default) (color 0 0 0 0))
-  )
   (wire (pts (xy 204.47 76.2) (xy 204.47 106.68))
     (stroke (width 0) (type default) (color 0 0 0 0))
@@
     (stroke (width 0) (type default) (color 0 0 0 0))
   )
+  (wire (pts (xy 124.46 82.55) (xy 121.92 82.55))
+    (stroke (width 0) (type default) (color 0 0 0 0))
+  )
   (wire (pts (xy 96.52 92.71) (xy 96.52 85.09))
     (stroke (width 0) (type default) (color 0 0 0 0))
@@
     (stroke (width 0) (type default) (color 0 0 0 0))
   )
-  (wire (pts (xy 121.92 82.55) (xy 121.92 85.09))
-    (stroke (width 0) (type default) (color 0 0 0 0))
-  )
   (wire (pts (xy 233.68 68.58) (xy 233.68 72.39))
     (stroke (width 0) (type default) (color 0 0 0 0))
@@
     (stroke (width 0) (type default) (color 0 0 0 0))
   )
-  (wire (pts (xy 97.79 109.22) (xy 132.08 109.22))
+  (wire (pts (xy 97.79 109.22) (xy 129.54 109.22))
     (stroke (width 0) (type default) (color 0 0 0 0))
   )
@@
     (stroke (width 0) (type default) (color 0 0 0 0))
   )
+  (wire (pts (xy 217.17 39.37) (xy 217.17 60.96))
+    (stroke (width 0) (type default) (color 0 0 0 0))
+  )
+  (wire (pts (xy 203.2 -38.1) (xy 203.2 -21.59))
+    (stroke (width 0) (type default) (color 0 0 0 0))
+  )
+  (wire (pts (xy 82.55 -6.35) (xy 116.84 -6.35))
+    (stroke (width 0) (type default) (color 0 0 0 0))
+  )
   (wire (pts (xy 132.08 109.22) (xy 213.36 109.22))
-    (stroke (width 0) (type default) (color 0 0 0 0))
-  )
-  (wire (pts (xy 217.17 39.37) (xy 217.17 60.96))
-    (stroke (width 0) (type default) (color 0 0 0 0))
-  )
-  (wire (pts (xy 203.2 -38.1) (xy 203.2 -21.59))
-    (stroke (width 0) (type default) (color 0 0 0 0))
-  )
-  (wire (pts (xy 82.55 -6.35) (xy 116.84 -6.35))
     (stroke (width 0) (type default) (color 0 0 0 0))
   )
@@
     (pin "1")
   )
-  (symbol (lib_id "power:GND") (at 121.92 93.98 0) (unit 1)
-    (in_bom yes) (on_board yes) (fields_autoplaced)
-    (property "Reference" "#PWR?" (id 0) (at 121.92 100.33 0)
-      (effects (font (size 1.27 1.27)) hide)
-    )
-    (property "Value" "GND" (id 1) (at 121.92 99.06 0))
-    (property "Footprint" "" (id 2) (at 121.92 93.98 0)
-      (effects (font (size 1.27 1.27)) hide)
-    )
-    (property "Datasheet" "" (id 3) (at 121.92 93.98 0)
-      (effects (font (size 1.27 1.27)) hide)
-    )
-    (pin "1")
-  )
   (symbol (lib_id "power:GND") (at 90.17 59.69 0) (unit 1)
     (in_bom yes) (on_board yes) (fields_autoplaced)
@@
     (pin "1")
   )
-  (symbol (lib_id "Device:R") (at 128.27 85.09 90) (unit 1)
-    (in_bom yes) (on_board yes) (fields_autoplaced)
-    (property "Reference" "R2" (id 0) (at 128.27 78.74 90))
-    (property "Value" "R" (id 1) (at 128.27 81.28 90))
-    (property "Footprint" "" (id 2) (at 128.27 86.868 90)
-      (effects (font (size 1.27 1.27)) hide)
-    )
-    (property "Datasheet" "~" (id 3) (at 128.27 85.09 0)
+  (symbol (lib_id "Device:R") (at 125.73 87.63 90) (unit 1)
+    (in_bom yes) (on_board yes) (fields_autoplaced)
+    (property "Reference" "R2" (id 0) (at 125.73 81.28 90))
+    (property "Value" "R" (id 1) (at 125.73 83.82 90))
+    (property "Footprint" "" (id 2) (at 125.73 89.408 90)
+      (effects (font (size 1.27 1.27)) hide)
+    )
+    (property "Datasheet" "~" (id 3) (at 125.73 87.63 0)
       (effects (font (size 1.27 1.27)) hide)
     )
@@
     (pin "9")
   )
+  (symbol (lib_id "power:GND") (at 124.46 82.55 0) (unit 1)
+    (in_bom yes) (on_board yes) (fields_autoplaced)
+    (property "Reference" "#PWR?" (id 0) (at 124.46 88.9 0)
+      (effects (font (size 1.27 1.27)) hide)
+    )
+    (property "Value" "GND" (id 1) (at 127 83.8199 0)
+      (effects (font (size 1.27 1.27)) (justify left))
+    )
+    (property "Footprint" "" (id 2) (at 124.46 82.55 0)
+      (effects (font (size 1.27 1.27)) hide)
+    )
+    (property "Datasheet" "" (id 3) (at 124.46 82.55 0)
+      (effects (font (size 1.27 1.27)) hide)
+    )
+    (pin "1")
+  )
   (sheet_instances
     (path "/" (page "1"))
@@
       (reference "#PWR?") (unit 1) (value "GND") (footprint "")
     )
-    (path "/8b7faa43-8807-43a1-b852-8a9a2586e698"
-      (reference "#PWR?") (unit 1) (value "GND") (footprint "")
-    )
     (path "/95975d8c-b8a8-427d-9744-0556356b7075"
       (reference "#PWR?") (unit 1) (value "GND") (footprint "")
@@
       (reference "#PWR?") (unit 1) (value "GND") (footprint "")
     )
+    (path "/fc8dfe5f-3578-40d2-986d-14b87d81e878"
+      (reference "#PWR?") (unit 1) (value "GND") (footprint "")
+    )
